File: adapter_board/panasonic_typewriter_interface/panasonic_typewriter_interface.kicad_sch (KiCad schematic)
At the start: 27 parts, among them J1 KMDGX-8S-AS, J2 Conn_02x03_Odd_Even, J4 Conn_01x06_MountingPin, J5 Conn_01x04_MountingPin, SW1 SW_SPDT, SW2 SW_Push

Commit message: misc updates
Parts:
- J3: value (none) -> Conn_01x06_MountingPin; symbol Connector_Generic_MountingPin:Conn_01x05_MountingPin -> Connector_Generic_MountingPin:Conn_01x06_MountingPin
- J4: value Conn_01x06_MountingPin -> (none); footprint Connector_JST:JST_GH_SM06B-GHS-TB_1x06-1MP_P1.25mm_Horizontal -> (none)
- J5: footprint (none) -> Connector_JST:JST_SH_SM04B-SRSS-TB_1x04-1MP_P1.00mm_Horizontal
Connections:
- net +5V: now also J3.5 (Pin_5)
- net GND: now also J3.6 (Pin_6); no longer J3.5 (Pin_5)
Changed lines of the file:
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@@
+    (stroke (width 0) (type default) (color 0 0 0 0))
+  )
+  (wire (pts (xy 27.94 143.51) (xy 39.37 143.51))
     (stroke (width 0) (type default) (color 0 0 0 0))
   )
@@
       (effects (font (size 1.27 1.27)) (justify left))
     )
-    (property "Footprint" "" (id 2) (at 92.71 142.24 0)
+    (property "Footprint" "Connector_JST:JST_SH_SM04B-SRSS-TB_1x04-1MP_P1.00mm_Horizontal" (id 2) (at 92.71 142.24 0)
       (effects (font (size 1.27 1.27)) hide)
     )
@@
     (pin "1")
   )
-  (symbol (lib_id "power:GND") (at 22.86 148.59 0) (unit 1)
-    (in_bom yes) (on_board yes) (fields_autoplaced)
-    (property "Reference" "#PWR0104" (id 0) (at 22.86 154.94 0)
-      (effects (font (size 1.27 1.27)) hide)
-    )
-    (property "Value" "GND" (id 1) (at 22.86 153.67 0))
-    (property "Footprint" "" (id 2) (at 22.86 148.59 0)
-      (effects (font (size 1.27 1.27)) hide)
-    )
-    (property "Datasheet" "" (id 3) (at 22.86 148.59 0)
+  (symbol (lib_id "power:GND") (at 22.86 151.13 0) (unit 1)
+    (in_bom yes) (on_board yes) (fields_autoplaced)
+    (property "Reference" "#PWR0104" (id 0) (at 22.86 157.48 0)
+      (effects (font (size 1.27 1.27)) hide)
+    )
+    (property "Value" "GND" (id 1) (at 22.86 156.21 0))
+    (property "Footprint" "" (id 2) (at 22.86 151.13 0)
+      (effects (font (size 1.27 1.27)) hide)
+    )
+    (property "Datasheet" "" (id 3) (at 22.86 151.13 0)
       (effects (font (size 1.27 1.27)) hide)
     )
@@
     (pin "2")
   )
-  (symbol (lib_id "power:GND") (at 27.94 143.51 0) (unit 1)
-    (in_bom yes) (on_board yes) (fields_autoplaced)
-    (property "Reference" "#PWR0107" (id 0) (at 27.94 149.86 0)
-      (effects (font (size 1.27 1.27)) hide)
-    )
-    (property "Value" "GND" (id 1) (at 27.94 148.59 0))
-    (property "Footprint" "" (id 2) (at 27.94 143.51 0)
-      (effects (font (size 1.27 1.27)) hide)
-    )
-    (property "Datasheet" "" (id 3) (at 27.94 143.51 0)
+  (symbol (lib_id "power:GND") (at 27.94 146.05 0) (unit 1)
+    (in_bom yes) (on_board yes) (fields_autoplaced)
+    (property "Reference" "#PWR0107" (id 0) (at 27.94 152.4 0)
+      (effects (font (size 1.27 1.27)) hide)
+    )
+    (property "Value" "GND" (id 1) (at 27.94 151.13 0))
+    (property "Footprint" "" (id 2) (at 27.94 146.05 0)
+      (effects (font (size 1.27 1.27)) hide)
+    )
+    (property "Datasheet" "" (id 3) (at 27.94 146.05 0)
       (effects (font (size 1.27 1.27)) hide)
     )
@@
     )
     (property "Datasheet" "" (id 3) (at 78.74 146.05 0)
+      (effects (font (size 1.27 1.27)) hide)
+    )
+    (pin "1")
+  )
+  (symbol (lib_id "power:+5V") (at 39.37 143.51 0) (unit 1)
+    (in_bom yes) (on_board yes) (fields_autoplaced)
+    (property "Reference" "#PWR0116" (id 0) (at 39.37 147.32 0)
+      (effects (font (size 1.27 1.27)) hide)
+    )
+    (property "Value" "+5V" (id 1) (at 39.37 138.43 0))
+    (property "Footprint" "" (id 2) (at 39.37 143.51 0)
+      (effects (font (size 1.27 1.27)) hide)
+    )
+    (property "Datasheet" "" (id 3) (at 39.37 143.51 0)
       (effects (font (size 1.27 1.27)) hide)
     )
@@
     (in_bom yes) (on_board yes)
     (property "Reference" "J4" (id 0) (at 57.15 132.08 0))
-    (property "Value" "Conn_01x06_MountingPin" (id 1) (at 67.31 133.35 0))
-    (property "Footprint" "Connector_JST:JST_GH_SM06B-GHS-TB_1x06-1MP_P1.25mm_Horizontal" (id 2) (at 57.15 140.97 0)
+    (property "Value" "" (id 1) (at 67.31 133.35 0))
+    (property "Footprint" "" (id 2) (at 57.15 140.97 0)
       (effects (font (size 1.27 1.27)) hide)
     )
@@
     (pin "1")
   )
-  (symbol (lib_id "Connector_Generic_MountingPin:Conn_01x05_MountingPin") (at 22.86 138.43 0) (mirror y) (unit 1)
+  (symbol (lib_id "Connector_Generic_MountingPin:Conn_01x06_MountingPin") (at 22.86 138.43 0) (mirror y) (unit 1)
     (in_bom yes) (on_board yes)
     (property "Reference" "J3" (id 0) (at 22.225 128.27 0))
-    (property "Value" "" (id 1) (at 33.02 130.81 0))
+    (property "Value" "Conn_01x06_MountingPin" (id 1) (at 44.45 129.54 0)
+      (effects (font (size 1.27 1.27)) (justify left))
+    )
     (property "Footprint" "" (id 2) (at 22.86 138.43 0)
       (effects (font (size 1.27 1.27)) hide)
@@
     (pin "4")
     (pin "5")
+    (pin "6")
     (pin "MP")
   )
@@
       (reference "#PWR0115") (unit 1) (value "GND") (footprint "")
     )
+    (path "/7924d673-38f7-46f2-a702-72b4b4c32c3c"
+      (reference "#PWR0116") (unit 1) (value "+5V") (footprint "")
+    )
     (path "/aa2ea573-3f20-43c1-aa99-1f9c6031a9aa"
       (reference "A1") (unit 1) (value "Arduino_Nano_v3.x") (footprint "Module:Arduino_Nano")
@@
     )
     (path "/bbc464fa-a92c-4a27-b6ac-d88919599829"
-      (reference "J3") (unit 1) (value "Conn_01x05_MountingPin") (footprint "Connector_JST:JST_GH_SM05B-GHS-TB_1x05-1MP_P1.25mm_Horizontal")
+      (reference "J3") (unit 1) (value "Conn_01x06_MountingPin") (footprint "Connector_JST:JST_GH_SM06B-GHS-TB_1x06-1MP_P1.25mm_Horizontal")
     )
     (path "/a68a461d-f4e8-469c-b958-a662712bd761"
