File: adapter_boards/panasonic_typewriter_interface/panasonic_typewriter_interface.kicad_sch (KiCad schematic)
At the start: 27 parts, among them J1 KMDGX-8S-AS, J2 Conn_02x03_Odd_Even, J3 Conn_01x06_MountingPin, J5 Conn_01x04_MountingPin, SW1 SW_SPDT, SW2 SW_Push

Commit message: Add fuse to main 5v rail; label unused IO pins; minor silkscreen mods
Parts:
- added F1: (no value), symbol Device:Polyfuse
- J3: footprint (none) -> Connector_JST:JST_GH_SM06B-GHS-TB_1x06-1MP_P1.25mm_Horizontal
- J4: value (none) -> Conn_01x06_MountingPin; footprint (none) -> Connector_JST:JST_GH_SM06B-GHS-TB_1x06-1MP_P1.25mm_Horizontal
Connections:
- net +5V: now also F1.1; no longer A1.27 (+5V)
- new net: A1.27 (+5V), F1.2
Changed lines of the file:
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@@
   (title_block
     (title "Panasonic Typewriter Interface")
-    (date "2024-08-29")
-    (rev "2024-08-A")
+    (date "2024-10-01")
+    (rev "2024-10-A")
     (company "github.com/xunker")
   )
@@
     (pin "2")
   )
+  (symbol (lib_id "Device:Polyfuse") (at 162.56 60.96 0) (unit 1)
+    (in_bom yes) (on_board yes) (fields_autoplaced)
+    (property "Reference" "F1" (id 0) (at 165.1 59.6899 0)
+      (effects (font (size 1.27 1.27)) (justify left))
+    )
+    (property "Value" "" (id 1) (at 165.1 62.2299 0)
+      (effects (font (size 1.27 1.27)) (justify left))
+    )
+    (property "Footprint" "" (id 2) (at 163.83 66.04 0)
+      (effects (font (size 1.27 1.27)) (justify left) hide)
+    )
+    (property "Datasheet" "~" (id 3) (at 162.56 60.96 0)
+      (effects (font (size 1.27 1.27)) hide)
+    )
+    (pin "1")
+    (pin "2")
+  )
   (symbol (lib_id "power:GND") (at 59.69 36.83 0) (unit 1)
     (in_bom yes) (on_board yes) (fields_autoplaced)
@@
     (in_bom yes) (on_board yes)
     (property "Reference" "J4" (id 0) (at 57.15 132.08 0))
-    (property "Value" "" (id 1) (at 67.31 133.35 0))
-    (property "Footprint" "" (id 2) (at 57.15 140.97 0)
+    (property "Value" "Conn_01x06_MountingPin" (id 1) (at 67.31 133.35 0))
+    (property "Footprint" "Connector_JST:JST_GH_SM06B-GHS-TB_1x06-1MP_P1.25mm_Horizontal" (id 2) (at 57.15 140.97 0)
       (effects (font (size 1.27 1.27)) hide)
     )
@@
       (effects (font (size 1.27 1.27)) (justify left))
     )
-    (property "Footprint" "" (id 2) (at 22.86 138.43 0)
+    (property "Footprint" "Connector_JST:JST_GH_SM06B-GHS-TB_1x06-1MP_P1.25mm_Horizontal" (id 2) (at 22.86 138.43 0)
       (effects (font (size 1.27 1.27)) hide)
     )
@@
     (pin "1")
   )
-  (symbol (lib_id "power:+5V") (at 162.56 64.77 0) (unit 1)
-    (in_bom yes) (on_board yes) (fields_autoplaced)
-    (property "Reference" "#PWR0108" (id 0) (at 162.56 68.58 0)
-      (effects (font (size 1.27 1.27)) hide)
-    )
-    (property "Value" "+5V" (id 1) (at 162.56 59.69 0))
-    (property "Footprint" "" (id 2) (at 162.56 64.77 0)
-      (effects (font (size 1.27 1.27)) hide)
-    )
-    (property "Datasheet" "" (id 3) (at 162.56 64.77 0)
+  (symbol (lib_id "power:+5V") (at 162.56 57.15 0) (unit 1)
+    (in_bom yes) (on_board yes) (fields_autoplaced)
+    (property "Reference" "#PWR0108" (id 0) (at 162.56 60.96 0)
+      (effects (font (size 1.27 1.27)) hide)
+    )
+    (property "Value" "+5V" (id 1) (at 162.56 52.07 0))
+    (property "Footprint" "" (id 2) (at 162.56 57.15 0)
+      (effects (font (size 1.27 1.27)) hide)
+    )
+    (property "Datasheet" "" (id 3) (at 162.56 57.15 0)
       (effects (font (size 1.27 1.27)) hide)
     )
@@
       (reference "D7") (unit 1) (value "LED") (footprint "LED_SMD:LED_0805_2012Metric")
     )
+    (path "/52949d6c-3d13-4c3f-aaae-0190262c1362"
+      (reference "F1") (unit 1) (value "Polyfuse") (footprint "Fuse:Fuse_1206_3216Metric")
+    )
     (path "/7140ec3e-8241-4c98-9305-3e76208507dc"

Commit message: Convert to kicad 8; add space for qr code
Parts:
- F1: value (none) -> Polyfuse; footprint (none) -> Fuse:Fuse_1206_3216Metric
